Commit message: removed unused leftness parameter and added hand_mesh_path parameter

File: urdf/hand.urdf.xacro (robot description, xacro)
@@ -1,8 +1,8 @@
 <?xml version="1.0"?>
 <robot xmlns:xacro="http://www.ros.org/wiki/xacro" name="hand">
+	<link name="hand"/>
 	<xacro:include filename="$(find soft_hand_description)/model/soft_hand.urdf.xacro"/>
-		<link name="hand"/>
-		<xacro:soft_hand parent="hand" name="gmu_hand" withAdaptiveTransmission="true" useMimicTag="true" left="$(arg leftness)">
-				<origin xyz="0.0 0.0 0.0" rpy="0 0 0"/>
-		</xacro:soft_hand>
+	<xacro:soft_hand parent="hand" name="gmu_hand" withAdaptiveTransmission="true" useMimicTag="true" left="false">
+		<origin xyz="0.0 0.0 0.0" rpy="0 0 0"/>
+	</xacro:soft_hand>
 </robot>

Commit message: added (commented out) parameter lines to use the pr2 gripper

File: urdf/hand.urdf.xacro (robot description, xacro)
@@ -6,3 +6,17 @@
 		<origin xyz="0.0 0.0 0.0" rpy="0 0 0"/>
 	</xacro:soft_hand>
+	<!-- <xacro:include filename="$(find pr2_description)/urdf/gripper_v0/gripper.urdf.xacro" />
+	<xacro:pr2_gripper_v0 reflect="-1.0" side="r" parent="hand"
+		screw_reduction="${4.0/1000.0}"
+		gear_ratio="${(729.0/25.0)*(22.0/16.0)}"
+		theta0="${3.6029*M_PI/180.0}"
+		phi0="${29.7089*M_PI/180.0}"
+		t0="${-0.1914/1000.0}"
+		L0="${37.5528/1000.0}"
+		h="${0.0/1000.0}"
+		a="${68.3698/1000.0}"
+		b="${43.3849/1000.0}"
+		r="${91.5/1000.0}" >
+		<origin xyz="0 0 0" rpy="0 0 0" />
+	</xacro:pr2_gripper_v0> -->
 </robot>
