Commit message: added table inside the GMU

File: grasp_modification_utility/urdf/hand.urdf.xacro (robot description, xacro)
@@ -20,3 +20,7 @@
 		<origin xyz="0 0 0" rpy="0 0 0" />
 	</xacro:pr2_gripper_v0> -->
+	<!-- <xacro:include filename="$(find dual_manipulation_grasp_db)/grasp_modification_utility/urdf/table.urdf.xacro"/>
+	<xacro:table parent="hand" name="table">
+		<origin xyz="0.0 0.0 0.0" rpy="0 0 0"/>
+	</xacro:table> -->
 </robot>
